Commit message: Add fingertip keypoints.

File: assets/hand_arm/robot/hand_arm.urdf (robot description, URDF)
Before this commit: robot hand_arm, 24 links, 23 joints
Links:
- added link index_fingertip
- added link little_fingertip
- added link middle_fingertip
- added link ring_fingertip
- added link thumb_fingertip
Joints:
- added joint if_distal_to_index_fingertip: type fixed, parent if_distal, child index_fingertip, origin xyz=-0.087 0.0175 0.041
- added joint lf_distal_to_little_fingertip: type fixed, parent lf_distal, child little_fingertip, origin xyz=0.064 0.0175 0.034
- added joint mf_distal_to_middle_fingertip: type fixed, parent mf_distal, child middle_fingertip, origin xyz=-0.0375 0.0175 0.049
- added joint rf_distal_to_ring_fingertip: type fixed, parent rf_distal, child ring_fingertip, origin xyz=0.014 0.0175 0.041
- added joint th_distal_to_thumb_fingertip: type fixed, parent th_distal, child thumb_fingertip, origin xyz=-0.023 0 0.015

Commit message: Save current state.

File: assets/hand_arm/robot/hand_arm.urdf (robot description, URDF)
Before this commit: robot hand_arm, 29 links, 28 joints
Links:
- link base_link_inertia: geometry visual mesh filename=meshes/ur5/visual/base.obj
- link wrist_3_link: geometry visual mesh filename=meshes/ur5/visual/wrist3.obj
