Commit message: Save changes.

File: assets/hand_arm/collision_boundaries/safety_walls_visible.urdf (robot description, URDF)
Before this commit: robot visible_collision_boundary, 1 links, 0 joints
Links:
- link base_link: geometry collision box size=.05 1.2 1.0; collision box size=.05 1.2 1.0

File: assets/hand_arm/collision_boundaries/table_offset_visible.urdf (robot description, URDF)
Before this commit: robot visible_table_offset, 1 links, 0 joints
Links:
- link base_link: geometry collision box size=.7 0.5 0.01

File: assets/hand_arm/easy_bin/bin.urdf (robot description, URDF)
Before this commit: robot easy_bin, 1 links, 0 joints
Links:
- link base_link: geometry collision box size=.015 .5 .125; collision box size=.015 .5 .125

File: assets/hand_arm/medium_bin/bin.urdf (robot description, URDF)
Before this commit: robot medium_bin, 1 links, 0 joints
Links:
- link base_link: geometry collision box size=.015 .35 .1; collision box size=.015 .35 .1

File: assets/hand_arm/robot/hand_arm_collision_is_visual.urdf (robot description, URDF)
Before this commit: robot hand_arm, 29 links, 28 joints
Joints:
- removed joint palm_to_if_proximal
- removed joint palm_to_mf_proximal
- removed joint palm_to_rf_proximal
- removed joint palm_to_th_proximal
- removed joint th_proximal_to_th_inter
- added joint index_finger: type revolute, parent palm, child if_proximal, origin xyz=0.0435 0 0.141, axis 1 0 0, limit lower=-1.571 upper=0.0 effort=0.75 velocity=2.09439510239
- added joint middle_finger: type revolute, parent palm, child mf_proximal, origin xyz=0.0187 0 0.141, axis 1 0 0, limit lower=-1.571 upper=0.0 effort=0.75 velocity=2.09439510239
- added joint ring_finger: type revolute, parent palm, child rf_proximal, origin xyz=-0.0069 0 0.134, axis 1 0 0, limit lower=-1.571 upper=0.0 effort=0.75 velocity=2.09439510239
- added joint thumb_flexion: type revolute, parent th_proximal, child th_inter, origin xyz=-0.024 0.005 0.001, axis 0 1 0, limit lower=0.0 upper=1.571 effort=0.75 velocity=2.09439510239
- added joint thumb_opposition: type revolute, parent palm, child th_proximal, origin xyz=-0.034 0.019 0.08, axis 0 0 1, limit lower=-1.571 upper=0.0 effort=0.75 velocity=2.09439510239
- joint if_proximal_to_if_distal: mimic joint=palm_to_if_proximal multiplier=1.0 -> joint=index_finger multiplier=1.0
- joint lf_proximal_to_lf_distal: mimic joint=palm_to_rf_proximal multiplier=1.0 -> joint=ring_finger multiplier=1.0
- joint mf_proximal_to_mf_distal: mimic joint=palm_to_mf_proximal multiplier=1.0 -> joint=middle_finger multiplier=1.0
- joint palm_to_lf_proximal: mimic joint=palm_to_rf_proximal multiplier=1.0 -> joint=ring_finger multiplier=1.0
- joint rf_proximal_to_rf_distal: mimic joint=palm_to_rf_proximal multiplier=1.0 -> joint=ring_finger multiplier=1.0
- joint th_inter_to_th_distal: mimic joint=th_proximal_to_th_inter multiplier=1.0 -> joint=thumb_flexion multiplier=1.0
